File: Esquemáticos/RemotePet/RemotePet.kicad_sch (KiCad schematic)
At the start: 7 parts

Commit message: Update esquemático con servos
Parts:
- added Food: (no value), symbol XFW-HX711:SERVO
- added Water: SERVO, symbol XFW-HX711:SERVO
- R1, R2: value (none) -> 1KΩ
- U1: value (none) -> ESP32_DevKit_V1_DOIT; footprint (none) -> ESP32_DevKit_V1_DOIT:esp32_devkit_v1_doit
- U2: value (none) -> xfw-hx711
- U3: value (none) -> Load_Cell
- U6: value (none) -> GY-30
- U?: value (none) -> WaterSensor
Connections:
- net IO25: now reaches U1.8 (IO25)
- net IO26: now reaches U1.9 (IO26)
Other:
- note added: "Servomotores"

Commit message: Sch-1
Parts:
- added 10uF1: 10uF, symbol Device:C
- added C1, C2: 0.22 uF, symbol Device:C
- added C3: 10uF, Capacitor_THT:CP_Radial_D4.0mm_P2.00mm, symbol Device:C
- added D1, D2: LED, symbol Device:LED
- added J1: USB_A, symbol Connector:USB_A
- added R3, R4: 1k, symbol Device:R
- added S1: EG1218, digikey-footprints:Switch_Slide_11.6x4mm_EG1218, symbol dk_Slide-Switches:EG1218
- added U5: L7805, symbol Regulator_Linear:L7805
- added U7: LM1117-3.3, symbol Regulator_Linear:LM1117-3.3
- added conexiones_entrada1: Conn_01x02_Male, symbol Connector:Conn_01x02_Male
- Food1: renamed from Food; value (none) -> SERVO; footprint (none) -> Connector_PinSocket_2.00mm:PinSocket_1x03_P2.00mm_Vertical
- U2: footprint (none) -> XFW
- U3: footprint (none) -> TerminalBlock_Phoenix:TerminalBlock_Phoenix_MKDS-1,5-3_1x03_P5.00mm_Horizontal
- U4: renamed from U?; footprint (none) -> Connector_PinSocket_2.00mm:PinSocket_1x03_P2.00mm_Vertical
- U6: footprint (none) -> Connector_PinSocket_2.00mm:PinSocket_1x05_P2.00mm_Vertical
- Water1: renamed from Water; footprint (none) -> Connector_PinSocket_2.00mm:PinSocket_1x03_P2.00mm_Vertical
Connections:
- net +3V3: now also C3.1, R3.2, U7.2 (VO)
- net +5V: now also Food1. (Vcc), U1.15 (VIN), U2. (VCC), U4. (VCC), U6. (VCC), Water1. (Vcc), C2.1, R4.2, U5.3 (OUT)
- net GND: now also Food1. (Vcc), U1.14 (GND), U2. (VCC), U4. (VCC), U6. (VCC), Water1. (Vcc), 10uF1.2, C1.2, C2.2, C3.2, D1.1 (K), D2.1 (K), J1.4 (GND), S1.3, U5.2 (GND), U7.1 (GND), conexiones_entrada1.2 (Pin_2)
- net IO18: now also U2. (VCC)
- net IO19: now also U2. (VCC)
- net IO2: now also U4. (VCC)
- net IO21: now also U6. (VCC)
- net IO22: now also U6. (VCC)
- net IO25: now also Food1. (Vcc)
- net IO26: now also Water1. (Vcc)
- net at R1.1: now also U2. (VCC), U3. (White)
- net at R1.2, R2.2: now also U2. (VCC)
- net at R2.1: now also U2. (VCC), U3. (White)
- net at U3. (White): now also U2. (VCC)
- new net: D2.2 (A), R4.1
- new net: D1.2 (A), R3.1
- new net v1: J1.1 (VBUS), S1.2, conexiones_entrada1.1 (Pin_1)
- new net vin: 10uF1.1, C1.1, S1.1, U5.1 (IN), U7.3 (VI)
- no-connect marks 0 -> 5
Other:
- moved on the sheet: U3

Commit message: SCH_finish
Parts:
- removed 10uF1: 10uF, symbol Device:C
- removed C1, C2: 0.22 uF, symbol Device:C
- removed C3: 10uF, Capacitor_THT:CP_Radial_D4.0mm_P2.00mm, symbol Device:C
- removed Food1, Water1: SERVO, Connector_PinSocket_2.00mm:PinSocket_1x03_P2.00mm_Vertical, symbol XFW-HX711:SERVO
- removed J1: USB_A, symbol Connector:USB_A
- removed U3: Load_Cell, TerminalBlock_Phoenix:TerminalBlock_Phoenix_MKDS-1,5-3_1x03_P5.00mm_Horizontal, symbol XFW-HX711:Load_Cell
- removed U4: WaterSensor, Connector_PinSocket_2.00mm:PinSocket_1x03_P2.00mm_Vertical, symbol XFW-HX711:WaterSensor
- removed U6: GY-30, Connector_PinSocket_2.00mm:PinSocket_1x05_P2.00mm_Vertical, symbol XFW-HX711:GY-30
- removed U7: LM1117-3.3, symbol Regulator_Linear:LM1117-3.3
- added C1, C2: 0.22 uF, Capacitor_THT:CP_Radial_D8.0mm_P5.00mm, symbol Device:C_Polarized
- added C3, C4: 10uF, Capacitor_THT:CP_Radial_D8.0mm_P5.00mm, symbol Device:C_Polarized
- added Esp32: Esp32_tx_rx, Connector_PinSocket_2.00mm:PinSocket_1x02_P2.00mm_Vertical, symbol Connector_Generic:Conn_01x02
- added Esp32Cam1: Esp32 Cam, Connector_PinSocket_2.00mm:PinSocket_1x02_P2.00mm_Vertical, symbol Connector_Generic:Conn_01x02
- added Food1: Servo1, Connector_PinSocket_2.00mm:PinSocket_1x03_P2.00mm_Vertical, symbol Connector:Conn_01x03_Female
- added Infrarroj6: MLX90614, Connector_PinSocket_2.00mm:PinSocket_1x04_P2.00mm_Vertical, symbol Connector_Generic:Conn_01x04
- added MotionS1: Motion Sensor, Connector_PinSocket_2.00mm:PinSocket_1x03_P2.00mm_Vertical, symbol Connector:Conn_01x03_Female
- added Screw1: Screw_Terminal_01x03, TerminalBlock_4Ucon:TerminalBlock_4Ucon_1x03_P3.50mm_Vertical, symbol Connector:Screw_Terminal_01x03
- added SensorSharp1, SensorSharp2: SensorSharp1, Connector_PinSocket_2.00mm:PinSocket_1x03_P2.00mm_Vertical, symbol Connector:Conn_01x03_Female
- added U4: LM1117-3.3, Package_TO_SOT_THT:TO-3P-3_Vertical, symbol Regulator_Linear:LM1117-3.3
- added U6: GY-30, Connector_PinSocket_2.00mm:PinSocket_1x05_P2.00mm_Vertical, symbol Connector_Generic:Conn_01x05
- added WaterS1, WaterS2: Water Sensor, Connector_PinSocket_2.00mm:PinSocket_1x03_P2.00mm_Vertical, symbol Connector:Conn_01x03_Female
- added water1: Servo2, Connector_PinSocket_2.00mm:PinSocket_1x03_P2.00mm_Vertical, symbol Connector:Conn_01x03_Female
- D1, D2: footprint (none) -> LED_THT:LED_D3.0mm_Clear
- R1, R2: footprint (none) -> Resistor_THT:R_Axial_DIN0309_L9.0mm_D3.2mm_P12.70mm_Horizontal
- R3, R4: value 1k -> 1KΩ; footprint (none) -> Resistor_THT:R_Axial_DIN0309_L9.0mm_D3.2mm_P12.70mm_Horizontal
- U2: footprint XFW -> Audio_Module:hx711
- U5: footprint (none) -> Package_TO_SOT_THT:TO-3P-3_Vertical
- conn_alimentación1: renamed from conexiones_entrada1; footprint (none) -> Connector_PinHeader_2.00mm:PinHeader_1x02_P2.00mm_Vertical
Connections:
- net +3V3: now also R3.1, C4.1, U4.2 (VO); no longer R3.2
- net +5V: now also R4.1, C2.1, Esp32Cam1.2 (Pin_2), Food1.1 (Pin_1), Infrarroj6.1 (Pin_1), MotionS1.3 (Pin_3), SensorSharp1.3 (Pin_3), SensorSharp2.3 (Pin_3), U6.5 (Pin_5), WaterS1.2 (Pin_2), WaterS2.2 (Pin_2), water1.1 (Pin_1); no longer R4.2
- net GND: now also C1.2, C2.2, C3.2, C4.2, Esp32Cam1.1 (Pin_1), Food1.2 (Pin_2), Infrarroj6.2 (Pin_2), MotionS1.1 (Pin_1), SensorSharp1.1 (Pin_1), SensorSharp2.1 (Pin_1), U4.1 (GND), U6.1 (Pin_1), U6.2 (Pin_2), WaterS1.1 (Pin_1), WaterS2.1 (Pin_1), water1.2 (Pin_2)
- net IO21: now also Infrarroj6.3 (Pin_3), U6.3 (Pin_3)
- net IO22: now also Infrarroj6.4 (Pin_4), U6.4 (Pin_4)
- net IO25: now also Food1.3 (Pin_3)
- net IO26: now also water1.3 (Pin_3)
- net at D2.2 (A): now also R4.2; no longer R4.1
- net at R1.1, U2. (VCC): now also R2.2
- net at D1.2 (A): now also R3.2; no longer R3.1
- net at R2.1, U2. (VCC): now also Screw1.3 (Pin_3)
- net IO27: now reaches U1.10 (IO27)
- net IO27: now also SensorSharp1.2 (Pin_2)
- net IO14: now reaches U1.11 (IO14)
- net IO14: now also SensorSharp2.2 (Pin_2)
- net IO12: now reaches U1.12 (IO12)
- net IO12: now also MotionS1.2 (Pin_2)
- net IO13: now reaches U1.13 (IO13)
- net IO13: now also WaterS2.3 (Pin_3)
- net TX_cam: now reaches U1.27 (RXD0/IO3)
- net TX_cam: now also Esp32.1 (Pin_1)
- net RX_cam: now reaches U1.28 (TXD0/IO1)
- net RX_cam: now also Esp32.2 (Pin_2)
- net IO35: now reaches U1.5 (IO35)
- net IO35: now also WaterS1.3 (Pin_3)
- net IO2: no longer names the net of U1.19 (IO2)
- net v1: no longer names the net of S1.2, conn_alimentación1.1 (Pin_1)
- net vin renamed VCC
- net VCC: now also C1.1, C3.1, U4.3 (VI)
- new net: R1.2, Screw1.1 (Pin_1), U2. (VCC)
- new net: Screw1.2 (Pin_2), U2. (VCC)
- no-connect marks 5 -> 15
Other:
- note added: "Light Sensor"
- note added: "Sensor Infrarrojo"
- note added: "Water Sensor"
- moved on the sheet: S1, conn_alimentación1
