File: Esquemáticos/RemotePet/RemotePet.kicad_pcb (KiCad board)
At the start: 2 copper layers, 1 part, among them U1 ESP32_DevKit_V1_DOIT

Commit message: Sch-1
Parts:
- added Food1: SERVO, Connector_PinSocket_2.00mm:PinSocket_1x03_P2.00mm_Vertical, F.Cu at (182.9, 61.0)
- added S1: EG1218, digikey-footprints:Switch_Slide_11.6x4mm_EG1218, F.Cu at (185.1, 56.2)
- added U3: Load_Cell, TerminalBlock_Phoenix:TerminalBlock_Phoenix_MKDS-1,5-3_1x03_P5.00mm_Horizontal, F.Cu at (167.3, 59.6)
- added U4: WaterSensor, Connector_PinSocket_2.00mm:PinSocket_1x03_P2.00mm_Vertical, F.Cu at (191.0, 61.0)
- added U6: GY-30, Connector_PinSocket_2.00mm:PinSocket_1x05_P2.00mm_Vertical, F.Cu at (114.3, 81.3)
- added Water1: SERVO, Connector_PinSocket_2.00mm:PinSocket_1x03_P2.00mm_Vertical, F.Cu at (186.9, 61.0)
Connections:
- U1 pad 14: unconnected-(U1-Pad14) -> GND
- U1 pad 15: unconnected-(U1-Pad15) -> 5V
- U1 pad 16: unconnected-(U1-Pad16) -> 3.3V
- U1 pad 17: unconnected-(U1-Pad17) -> GND
- U1 pad 19: unconnected-(U1-Pad19) -> IO2
- U1 pad 24: unconnected-(U1-Pad24) -> IO18
- U1 pad 25: unconnected-(U1-Pad25) -> IO19
- U1 pad 26: unconnected-(U1-Pad26) -> IO21
- U1 pad 29: unconnected-(U1-Pad29) -> IO22
- U1 pad 8: unconnected-(U1-Pad8) -> IO25
- U1 pad 9: unconnected-(U1-Pad9) -> IO26

Commit message: SCH_finish
Parts:
- removed U3: Load_Cell, TerminalBlock_Phoenix:TerminalBlock_Phoenix_MKDS-1,5-3_1x03_P5.00mm_Horizontal
- removed Water1: SERVO, Connector_PinSocket_2.00mm:PinSocket_1x03_P2.00mm_Vertical
- added C1: 0.22 uF, Capacitor_THT:CP_Radial_D8.0mm_P5.00mm, F.Cu at (182.9, 97.8)
- added C2: 0.22 uF, Capacitor_THT:CP_Radial_D8.0mm_P5.00mm, F.Cu at (199.9, 84.2)
- added C3: 10uF, Capacitor_THT:CP_Radial_D8.0mm_P5.00mm, F.Cu at (192.6, 97.8)
- added C4: 10uF, Capacitor_THT:CP_Radial_D8.0mm_P5.00mm, F.Cu at (211.7, 80.2)
- added D1: LED, LED_THT:LED_D3.0mm_Clear, F.Cu at (209.7, 95.8)
- added D2: LED, LED_THT:LED_D3.0mm_Clear, F.Cu at (224.7, 80.7)
- added Esp32: Esp32_tx_rx, Connector_PinSocket_2.00mm:PinSocket_1x02_P2.00mm_Vertical, F.Cu at (217.3, 88.0)
- added Esp32Cam1: Esp32 Cam, Connector_PinSocket_2.00mm:PinSocket_1x02_P2.00mm_Vertical, F.Cu at (232.5, 71.9)
- added Infrarroj6: MLX90614, Connector_PinSocket_2.00mm:PinSocket_1x04_P2.00mm_Vertical, F.Cu at (178.4, 95.0)
- added MotionS1: Motion Sensor, Connector_PinSocket_2.00mm:PinSocket_1x03_P2.00mm_Vertical, F.Cu at (213.3, 87.0)
- added R1: 1KΩ, Resistor_THT:R_Axial_DIN0309_L9.0mm_D3.2mm_P12.70mm_Horizontal, F.Cu at (177.9, 85.9)
- added R2: 1KΩ, Resistor_THT:R_Axial_DIN0309_L9.0mm_D3.2mm_P12.70mm_Horizontal, F.Cu at (195.0, 77.0)
- added R3: 1KΩ, Resistor_THT:R_Axial_DIN0309_L9.0mm_D3.2mm_P12.70mm_Horizontal, F.Cu at (195.0, 72.3)
- added R4: 1KΩ, Resistor_THT:R_Axial_DIN0309_L9.0mm_D3.2mm_P12.70mm_Horizontal, F.Cu at (177.9, 90.6)
- added Screw1: Screw_Terminal_01x03, TerminalBlock_4Ucon:TerminalBlock_4Ucon_1x03_P3.50mm_Vertical, F.Cu at (96.8, 61.8)
- added SensorSharp1: SensorSharp1, Connector_PinSocket_2.00mm:PinSocket_1x03_P2.00mm_Vertical, F.Cu at (224.4, 71.9)
- added SensorSharp2: SensorSharp1, Connector_PinSocket_2.00mm:PinSocket_1x03_P2.00mm_Vertical, F.Cu at (209.2, 87.0)
- added U2: xfw-hx711, Audio_Module:hx711, F.Cu at (182.9, 114.3)
- added U5: L7805, Package_TO_SOT_THT:TO-3P-3_Vertical, F.Cu at (179.4, 73.7)
- added WaterS1: Water Sensor, Connector_PinSocket_2.00mm:PinSocket_1x03_P2.00mm_Vertical, F.Cu at (228.5, 71.9)
- added WaterS2: Water Sensor, Connector_PinSocket_2.00mm:PinSocket_1x03_P2.00mm_Vertical, F.Cu at (206.0, 95.1)
- added conn_alimentación1: Conn_01x02_Male, Connector_PinHeader_2.00mm:PinHeader_1x02_P2.00mm_Vertical, F.Cu at (201.9, 99.0)
- added water1: Servo2, Connector_PinSocket_2.00mm:PinSocket_1x03_P2.00mm_Vertical, F.Cu at (221.0, 80.0)
- Food1: value SERVO -> Servo1
- U4: value WaterSensor -> LM1117-3.3; footprint Connector_PinSocket_2.00mm:PinSocket_1x03_P2.00mm_Vertical -> Package_TO_SOT_THT:TO-3P-3_Vertical
- moved U6 81.1 mm to (195.4, 81.4)
- moved Food1 35.6 mm to (201.9, 91.0)
- moved S1 32.9 mm to (213.5, 72.7)
- moved U4 22.7 mm to (179.4, 80.5)
Connections:
- Food1 pad 1: (no net) -> 5V
- Food1 pad 2: (no net) -> GND
- Food1 pad 3: (no net) -> IO25
- S1 pad 1: vin -> VCC
- S1 pad 2: /v1 -> Net-(S1-Pad2)
- U1 pad 10: unconnected-(U1-Pad10) -> IO27
- U1 pad 11: unconnected-(U1-Pad11) -> IO14
- U1 pad 12: unconnected-(U1-Pad12) -> IO12
- U1 pad 13: unconnected-(U1-Pad13) -> IO13
- U1 pad 19: IO2 -> unconnected-(U1-Pad19)
- U1 pad 27: unconnected-(U1-Pad27) -> TX_cam
- U1 pad 28: unconnected-(U1-Pad28) -> RX_cam
- U1 pad 5: unconnected-(U1-Pad5) -> IO35
- U4 pad 1: (no net) -> GND
- U4 pad 2: (no net) -> 3.3V
- U4 pad 3: (no net) -> VCC
- U6 pad 1: (no net) -> GND
- U6 pad 2: (no net) -> GND
- U6 pad 3: (no net) -> IO21
- U6 pad 4: (no net) -> IO22
- U6 pad 5: (no net) -> 5V

Commit message: PCB-FINISH
Parts:
- C1, C2, C3, C4: footprint Capacitor_THT:CP_Radial_D8.0mm_P5.00mm -> Capacitor_THT:CP_Radial_D4.0mm_P2.00mm
- U4, U5: footprint Package_TO_SOT_THT:TO-3P-3_Vertical -> Package_TO_SOT_THT:TO-220-3_Vertical
- moved SensorSharp1 115.6 mm to (119.9, 121.3), turned to 90 degrees
- moved D2 110.7 mm to (115.2, 65.1), turned to -90 degrees
- moved S1 109.4 mm to (104.1, 76.0), turned to 90 degrees
- moved SensorSharp2 109.2 mm to (105.5, 121.3), turned to 90 degrees
- moved C4 109.0 mm to (104.1, 97.8), turned to 90 degrees
- moved conn_alimentación1 108.1 mm to (97.8, 69.8)
- moved Esp32Cam1 103.1 mm to (130.2, 59.3), turned to 90 degrees
- moved C2 96.3 mm to (103.8, 90.2), turned to 90 degrees
- moved D1 96.3 mm to (114.6, 111.2), turned to 90 degrees
- moved WaterS1 89.3 mm to (154.1, 121.3), turned to 90 degrees
- moved C3 88.6 mm to (104.1, 102.9), turned to -90 degrees
- moved Esp32 86.1 mm to (136.2, 59.2), turned to 90 degrees
- moved U4 84.7 mm to (96.5, 97.8), turned to -90 degrees
- moved U5 83.5 mm to (96.5, 83.8), turned to -90 degrees
- moved R3 82.4 mm to (114.8, 91.7), turned to -90 degrees
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Connections:
- R1 pad 1: Net-(U2-Pad)_1 -> Net-(R1-Pad1)
- R1 pad 2: Net-(Screw1-Pad1) -> Net-(R1-Pad2)
- R2 pad 1: Net-(Screw1-Pad3) -> Net-(R2-Pad1)
- R2 pad 2: Net-(U2-Pad)_1 -> Net-(R1-Pad1)
- Screw1 pad 1: Net-(Screw1-Pad1) -> Net-(R1-Pad2)
- Screw1 pad 2: Net-(U2-Pad) -> Net-(Screw1-Pad2)
- Screw1 pad 3: Net-(Screw1-Pad3) -> Net-(R2-Pad1)
Routing:
- net IO26: track 0.00 -> 96.8 mm, vias 0 -> 1
- net 3.3V: track 0.00 -> 70.3 mm
- net IO35: track 0.00 -> 60.4 mm
- net IO27: track 0.00 -> 54.6 mm
- net IO25: track 0.00 -> 50.1 mm, vias 0 -> 1
- net Net-(R2-Pad1): track 0.00 -> 48.9 mm
- net IO18: track 0.00 -> 48.5 mm
- net IO19: track 0.00 -> 43.7 mm
- net VCC: track 0.00 -> 42.1 mm
- net IO14: track 0.00 -> 34.6 mm
- net IO12: track 0.00 -> 34.4 mm
- net Net-(R1-Pad2): track 0.00 -> 30.6 mm
- net Net-(Screw1-Pad2): track 0.00 -> 28.3 mm
- net TX_cam: track 0.00 -> 27.0 mm
- net IO13: track 0.00 -> 26.4 mm
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- added copper zone on F.Cu, net 5V
- added copper zone on B.Cu, net GND
Other:
- board outline added: 87.2 x 72.6 mm
